File: LAN.kicad_sch (KiCad schematic)
At the start: 54 parts, among them U3 W5500, U4 0826-1X1T-KL-F, U6 Ag5810, Y1 XO32F025000GEHE001

Commit message: fix: crystal clock enable pin to 3v3
Parts:
- removed R6: 1M, Resistor_SMD:R_0603_1608Metric, symbol Device:R
Connections:
- net +3.3V: now also C31.2, Y1.1 (TRI_STATE)
- net XO: no longer C31.2, Y1.1 (TRI_STATE)
Changed lines of the file:
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@@
 	)
 	(junction
+		(at 25.4 168.91)
+		(diameter 0)
+		(color 0 0 0 0)
+	)
+	(junction
 		(at 105.41 29.21)
 		(diameter 0)
@@
 	)
 	(junction
-		(at 25.4 168.91)
-		(diameter 0)
-		(color 0 0 0 0)
-	)
-	(junction
 		(at 60.96 170.18)
 		(diameter 0)
@@
 	)
 	(junction
-		(at 25.4 149.86)
-		(diameter 0)
-		(color 0 0 0 0)
-	)
-	(junction
 		(at 138.43 157.48)
 		(diameter 0)
@@
 	)
 	(junction
-		(at 60.96 149.86)
-		(diameter 0)
-		(color 0 0 0 0)
-	)
-	(junction
 		(at 257.81 156.21)
 		(diameter 0)
@@
 	(wire
 		(pts
-			(xy 60.96 146.05) (xy 60.96 149.86)
-		)
-		(stroke
-			(width 0)
-			(type default)
-		)
-	)
-	(wire
-		(pts
 			(xy 33.02 158.75) (xy 29.21 158.75)
 		)
@@
 	(wire
 		(pts
-			(xy 25.4 146.05) (xy 25.4 149.86)
-		)
-		(stroke
-			(width 0)
-			(type default)
-		)
-	)
-	(wire
-		(pts
 			(xy 36.83 76.2) (xy 48.26 76.2)
 		)
@@
 	(wire
 		(pts
-			(xy 60.96 149.86) (xy 60.96 162.56)
+			(xy 60.96 146.05) (xy 60.96 162.56)
 		)
 		(stroke
@@
 	(wire
 		(pts
-			(xy 46.99 149.86) (xy 60.96 149.86)
-		)
-		(stroke
-			(width 0)
-			(type default)
-		)
-	)
-	(wire
-		(pts
 			(xy 229.87 153.67) (xy 234.95 153.67)
 		)
@@
 	(wire
 		(pts
+			(xy 29.21 158.75) (xy 25.4 158.75)
+		)
+		(stroke
+			(width 0)
+			(type default)
+		)
+	)
+	(wire
+		(pts
 			(xy 25.4 168.91) (xy 25.4 173.99)
 		)
@@
 	(wire
 		(pts
-			(xy 25.4 149.86) (xy 25.4 168.91)
-		)
-		(stroke
-			(width 0)
-			(type default)
-		)
-	)
-	(wire
-		(pts
 			(xy 66.04 101.6) (xy 66.04 109.22)
 		)
@@
 	(wire
 		(pts
-			(xy 109.22 135.89) (xy 93.98 135.89)
+			(xy 25.4 158.75) (xy 25.4 168.91)
 		)
 		(stroke
@@
 	(wire
 		(pts
-			(xy 138.43 135.89) (xy 138.43 137.16)
+			(xy 109.22 135.89) (xy 93.98 135.89)
 		)
 		(stroke
@@
 	(wire
 		(pts
-			(xy 92.71 29.21) (xy 99.06 29.21)
+			(xy 138.43 135.89) (xy 138.43 137.16)
 		)
 		(stroke
@@
 	(wire
 		(pts
-			(xy 168.91 25.4) (xy 168.91 29.21)
+			(xy 92.71 29.21) (xy 99.06 29.21)
 		)
 		(stroke
@@
 	(wire
 		(pts
-			(xy 25.4 149.86) (xy 39.37 149.86)
+			(xy 168.91 25.4) (xy 168.91 29.21)
 		)
 		(stroke
@@
 		)
 	)
-	(label "XO"
-		(at 25.4 146.05 0)
-		(effects
-			(font
-				(size 1.27 1.27)
-			)
-			(justify left bottom)
-		)
-	)
 	(label "LAN.SCLK"
 		(at 36.83 48.26 0)
@@
 					(unit 1)
 				)
-			)
-		)
-	)
-	(symbol
-		(lib_id "Device:R")
-		(at 43.18 149.86 90)
-		(unit 1)
-		(exclude_from_sim no)
-		(in_bom yes)
-		(on_board yes)
-		(dnp no)
-		(property "Reference" "R6"
-			(at 43.18 149.86 90)
-			(effects
-				(font
-					(size 1.27 1.27)
-				)
-			)
-		)
-		(property "Value" "1M"
-			(at 43.18 146.05 90)
-			(effects
-				(font
-					(size 1.27 1.27)
-				)
-			)
-		)
-		(property "Footprint" "Resistor_SMD:R_0603_1608Metric"
-			(at 43.18 151.638 90)
-			(effects
-				(font
-					(size 1.27 1.27)
-				)
-				(hide yes)
-			)
-		)
-		(property "Datasheet" "https://jlcpcb.com/api/file/downloadByFileSystemAccessId/8588898610864410624"
-			(at 43.18 149.86 0)
-			(effects
-				(font
-					(size 1.27 1.27)
-				)
-				(hide yes)
-			)
-		)
-		(property "Description" "100mW Thick Film Resistors 75V ±100ppm/℃ ±1% 1MΩ 0603 Chip Resistor - Surface Mount ROHS"
-			(at 43.18 149.86 0)
-			(effects
-				(font
-					(size 1.27 1.27)
-				)
-				(hide yes)
-			)
-		)
-		(property "Manufacturer" "YAGEO"
-			(at 43.18 149.86 90)
-			(effects
-				(font
-					(size 1.27 1.27)
-				)
-				(hide yes)
-			)
-		)
-		(property "MPN" "RC0603FR-071ML"
-			(at 43.18 149.86 90)
-			(effects
-				(font
-					(size 1.27 1.27)
-				)
-				(hide yes)
-			)
-		)
-		(property "JLCPCB Part #" "C105578"
-			(at 43.18 149.86 90)
-			(effects
-				(font
-					(size 1.27 1.27)
-				)
-				(hide yes)
-			)
-		)
-		(pin "1"
-		)
-		(pin "2"
-		)
-		(instances
-			(project ""
-				(path "/76f3fa83-72cd-42e5-a695-3afc9e289467/7a59ef83-1c1e-4921-8744-eadb3652d7d5"
-					(reference "R6")
-					(unit 1)
-				)
