File: LAN.kicad_sch (KiCad schematic)
At the start: 53 parts, among them U3 W5500, U4 0826-1X1T-KL-F, U6 Ag5810, Y1 XO32F025000GEHE001

Commit message: fix: specify 25V rating on caps on the 12V rail (#3)
Parts:
- C43, C44: value 1000u -> 1000u 25V
Changed lines of the file:
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@@
 			)
 		)
-		(property "Value" "1000u"
+		(property "Value" "1000u 25V"
 			(at 239.268 154.94 0)
 			(effects
@@
 			)
 		)
-		(property "Value" "1000u"
+		(property "Value" "1000u 25V"
 			(at 239.522 144.78 0)
 			(effects
