File: SqueezeAMPPOE.kicad_pcb (KiCad board)
At the start: 4 copper layers, 140 x 81 mm, 116 parts, among them J1 Conn_01x04_Pin, J2 Conn_01x02_Pin, J3 Screw_Terminal_01x02, J4 Screw_Terminal_01x02, SW1 SW_Push, U1 ESP32-WROVER-E-N4R8, U2 TAS5756MDCAR, U3 W5500, U4 0826-1X1T-KL-F, U6 Ag5810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

Commit message: fix: crystal clock enable pin to 3v3
Parts:
- removed R6: 1M, Resistor_SMD:R_0603_1608Metric
Connections:
- C31 pad 2: /LAN/XO -> +3.3V
- Y1 pad 1: /LAN/XO -> +3.3V
Routing:
- net /LAN/CLKIN: track 24.6 -> 12.2 mm
- net /LAN/XO: track 6.56 -> 0.00 mm
- net +3.3V: track 279.9 -> 286.3 mm
