File: SqueezeAMPPOE.kicad_pcb (KiCad board)
At the start: 4 copper layers, 140 x 81 mm, 115 parts, among them J1 Conn_01x04_Pin, J2 Conn_01x02_Pin, J3 Screw_Terminal_01x02, J4 Screw_Terminal_01x02, SW1 SW_Push, U1 ESP32-WROVER-E-N4R8, U2 TAS5756MDCAR, U3 W5500, U4 0826-1X1T-KL-F, U6 Ag5810, U7 TPS56339DDCR, Y1 XO32F025000GEHE001

Commit message: fix: specify 25V rating on caps on the 12V rail (#3)
Parts:
- C13, C15, C5, C6: value 10u -> 10u 25V
- C43, C44, C45, C46: value 1000u -> 1000u 25V
Changed lines of the file:
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@@
 			)
 		)
-		(property "Value" "1000u"
+		(property "Value" "1000u 25V"
 			(at 0 6.3 90)
 			(layer "F.Fab")
@@
 			)
 		)
-		(property "Value" "1000u"
+		(property "Value" "1000u 25V"
 			(at 0 6.3 0)
 			(layer "F.Fab")
@@
 			)
 		)
-		(property "Value" "1000u"
+		(property "Value" "1000u 25V"
 			(at 0 6.3 0)
 			(layer "F.Fab")
@@
 			)
 		)
-		(property "Value" "1000u"
+		(property "Value" "1000u 25V"
 			(at 0 6.3 90)
 			(layer "F.Fab")
@@
 			)
 		)
-		(property "Value" "10u"
+		(property "Value" "10u 25V"
 			(at 0 1.43 90)
 			(layer "F.Fab")
@@
 			)
 		)
-		(property "Value" "10u"
+		(property "Value" "10u 25V"
 			(at 0 1.43 90)
 			(layer "F.Fab")
@@
 			)
 		)
-		(property "Value" "10u"
+		(property "Value" "10u 25V"
 			(at 0 1.43 90)
 			(layer "F.Fab")
@@
 			)
 		)
-		(property "Value" "10u"
+		(property "Value" "10u 25V"
 			(at 0 1.43 90)
 			(layer "F.Fab")
