File: AMP.kicad_sch (KiCad schematic)
At the start: 33 parts, among them J3 Screw_Terminal_01x02, J4 Screw_Terminal_01x02, U2 TAS5756MDCAR

Commit message: fix: specify 25V rating on caps on the 12V rail (#3)
Parts:
- C13, C15: value 10u -> 10u 25V
- C45, C46: value 1000u -> 1000u 25V
Changed lines of the file:
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@@
 			)
 		)
-		(property "Value" "1000u"
+		(property "Value" "1000u 25V"
 			(at 96.012 27.94 0)
 			(effects
@@
 			)
 		)
-		(property "Value" "10u"
+		(property "Value" "10u 25V"
 			(at 123.19 27.94 0)
 			(effects
@@
 			)
 		)
-		(property "Value" "10u"
+		(property "Value" "10u 25V"
 			(at 115.57 27.94 0)
 			(effects
@@
 			)
 		)
-		(property "Value" "1000u"
+		(property "Value" "1000u 25V"
 			(at 106.172 27.94 0)
 			(effects
